Commit message: palm link changed to base link

File: schunk_ezn64/urdf/ezn64.urdf.xacro (robot description, xacro)
@@ -3,13 +3,13 @@
     <xacro:macro name="schunk_ezn64" params="parent name *origin ">
 <!--       PALM -->
-      <joint name="${name}_palm_joint" type="fixed" >
+      <joint name="${name}_base_joint" type="fixed" >
 	<parent link="${parent}" />
-	<child link="${name}_palm_link" />
+	<child link="${name}_base_link" />
 	<xacro:insert_block name="origin" />
       </joint>
-      <link name="${name}_palm_link">
+      <link name="${name}_base_link">
 	  <visual>
              <geometry>
-                <mesh filename="package://ezn64/meshes/ezn64_palm_link.STL" />
+                <mesh filename="package://schunk_ezn64/meshes/ezn64_base_link.STL" />
              </geometry>
              <material name="silver">
@@ -19,5 +19,5 @@
 	  <collision>
             <geometry>
-               <mesh filename="package://ezn64/meshes/ezn64_palm_link.STL" />
+               <mesh filename="package://schunk_ezn64/meshes/ezn64_base_link.STL" />
 	    </geometry>
 	    <material name="black">
@@ -28,5 +28,5 @@
 <!--       FINGER 1 -->
       <joint name="${name}_finger_1_joint" type="prismatic" >
-	<parent link="${name}_palm_link" />
+	<parent link="${name}_base_link" />
 	<child link="${name}_finger_1_link" />
 	<limit effort="0" lower="0" upper="0.006" velocity="0"/>
@@ -37,5 +37,5 @@
 	<visual>
 	  <geometry>
-	    <mesh filename="package://ezn64/meshes/ezn64_finger_1.STL" />
+	    <mesh filename="package://schunk_ezn64/meshes/ezn64_finger_1.STL" />
 	  </geometry>
 	    <material name="black"/>
@@ -43,5 +43,5 @@
 	<collision>
 	  <geometry>
-	    <mesh filename="package://ezn64/meshes/ezn64_finger_1.STL" />
+	    <mesh filename="package://schunk_ezn64/meshes/ezn64_finger_1.STL" />
 	  </geometry>
 	    <material name="black" />
@@ -51,5 +51,5 @@
       <joint name="${name}_finger_2_joint" type="prismatic" >
 	<mimic joint="${name}_finger_1_joint" multiplier="1" offset="0"/>
-	<parent link="${name}_palm_link" />
+	<parent link="${name}_base_link" />
 	<child link="${name}_finger_2_link" />
 	<limit effort="0" lower="0" upper="0.006" velocity="0"/>
@@ -60,5 +60,5 @@
 	<visual>
 	  <geometry>
-	    <mesh filename="package://ezn64/meshes/ezn64_finger_2.STL" />
+	    <mesh filename="package://schunk_ezn64/meshes/ezn64_finger_2.STL" />
 	  </geometry>
 	    <material name="black"/>
@@ -66,5 +66,5 @@
 	<collision>
 	  <geometry>
-	    <mesh filename="package://ezn64/meshes/ezn64_finger_2.STL" />
+	    <mesh filename="package://schunk_ezn64/meshes/ezn64_finger_2.STL" />
 	  </geometry>
 	    <material name="black" />
@@ -74,5 +74,5 @@
       <joint name="${name}_finger_3_joint" type="prismatic" >
 	<mimic joint="${name}_finger_1_joint" multiplier="1" offset="0"/>
-	<parent link="${name}_palm_link" />
+	<parent link="${name}_base_link" />
 	<child link="${name}_finger_3_link" />
 	<limit effort="0" lower="0" upper="0.006" velocity="0"/>
@@ -83,5 +83,5 @@
 	<visual>
 	  <geometry>
-	    <mesh filename="package://ezn64/meshes/ezn64_finger_3.STL" />
+	    <mesh filename="package://schunk_ezn64/meshes/ezn64_finger_3.STL" />
 	  </geometry>
 	    <material name="black"/>
@@ -89,5 +89,5 @@
 	<collision>
 	  <geometry>
-	    <mesh filename="package://ezn64/meshes/ezn64_finger_3.STL" />
+	    <mesh filename="package://schunk_ezn64/meshes/ezn64_finger_3.STL" />
 	  </geometry>
 	    <material name="black" />
